Commit message: offline planning ok

File: motomini/urdf/custom_object.urdf.xacro (robot description, xacro)
@@ -1,7 +1,7 @@
 <?xml version="1.0"?>
 <robot xmlns:xacro="http://www.ros.org/wiki/xacro" name="target_object">
-    <xacro:arg name="mesh_path" default="package://motomini/meshes/puzzel.stl" />
+    <xacro:arg name="mesh_path" default="package://motomini/meshes/puzzel_mount.stl" />
     <xacro:arg name="gravity_off" default="true" />
-    <xacro:arg name="mesh_scale" default="0.001" />
+    <xacro:arg name="mesh_scale" default="1.0" />
     <link name="object_link">
         <visual>

File: motomini/urdf/motoman_motomini.urdf (robot description, URDF)
Before this commit: robot motoman_motomini, 10 links, 9 joints
Links:
- link workcell: geometry visual mesh filename=package://motomini/meshes/workcell.stl scale=0.001 0.001 0.001

File: motomini/urdf/motoman_motomini_sensors.urdf.xacro (robot description, xacro)
@@ -37,5 +37,5 @@
         <parent link="workcell" />
         <child link="world_depth_camera_link" />
-        <origin xyz="-0.2 -0.2 0.25" rpy="0 1.57142857143 0" />
+        <origin xyz="0.225 -0.225 0.245" rpy="0 3.14159 3.14159" />
     </joint>
     <gazebo reference="world_depth_camera_link">
