Commit message: [bug] dodge bu stuck

File: motomini/urdf/motoman_motomini_wrapper_realbot.urdf.xacro (robot description, xacro)
@@ -14,4 +14,5 @@
     <xacro:include filename="motoman_motomini_tool.xacro" />
     <xacro:include filename="2axis.urdf.xacro" />
+    <xacro:include filename="obstacle.urdf.xacro" />
     <!-- <xacro:include filename="plate.urdf.xacro" /> -->
     <!-- ========= TOOLS ========= -->
@@ -30,4 +31,10 @@
         <child link="gantry_base_link" />
         <origin xyz="0.03 -0.46 0.0602" rpy="0 0 3.14" />
+    </joint>
+    <!-- Obstacle joint (position controlled by obstacle_simulator TF broadcaster) -->
+    <joint name="world_to_obstacle" type="fixed">
+        <parent link="world" />
+        <child link="obstacle_link" />
+        <origin xyz="0.1 0.0 0.15" rpy="0 0 0" />
     </joint>
     <!-- <joint name="world_to_plate" type="fixed">

File: robot_planning/urdf/motoman_motomini.urdf (robot description, URDF)
Before this commit: robot motoman_motomini, 10 links, 9 joints
Links:
- added link obstacle_link; collision cylinder length=0.05 radius=0.02
Joints:
- added joint world_to_obstacle: type fixed, parent world, child obstacle_link, origin xyz=0.1 0.0 0.2 rpy=0 0 0
