Commit message: [bug] colision, before adding OLM

File: motomini/urdf/motoman_motomini.urdf (robot description, URDF)
Before this commit: robot motoman_motomini, 10 links, 9 joints
Links:
- link workcell: geometry collision mesh filename=package://motomini/meshes/workcell.stl scale=0.001 0.001 0.001; visual mesh filename=package://motomini/meshes/workcell.stl scale=0.001 0.001 0.001

File: motomini/urdf/motoman_motomini_wrapper.urdf.xacro (robot description, xacro)
@@ -1,10 +1,20 @@
 <?xml version="1.0" encoding="utf-8"?>
-<robot xmlns:xacro="http://www.ros.org/wiki/xacro" name="motoman_motomini">
+<robot name="motoman_motomini"
+    xmlns:xacro="http://www.ros.org/wiki/xacro"
+    xmlns:tesseract="http://ros.org/wiki/tesseract"
+    tesseract:make_convex="true">
     <!-- ========= ARG FIRST ========= -->
     <xacro:arg name="controllers_file" default="" />
     <xacro:property name="controllers_file" value="$(arg controllers_file)" />
+    <xacro:arg name="tool_type" default="gripper" />
+    <xacro:property name="tool_type" value="$(arg tool_type)" />
     <!-- ========= INCLUDE ROBOT ========= -->
     <xacro:include filename="motoman_motomini.urdf" />
     <xacro:include filename="motoman_motomini_sensors.urdf.xacro" />
+    <xacro:include filename="motoman_motomini_tool.xacro" />
+    <!-- ========= TOOLS ========= -->
+    <xacro:motomini_tool
+        parent_link="tool0"
+        tool_type="${tool_type}" />
     <!-- ========= WORLD FIX ========= -->
     <link name="world" />

File: robot_model/urdf/motomini_macro_no_world.xacro (robot description, xacro)
@@ -2,22 +2,21 @@
 <robot xmlns:xacro="http://ros.org/wiki/xacro">
   <xacro:macro name="motoman_motomini" params="prefix">
-    <material name="yaskawa_blue">
-      <color rgba="0.12941 0.14902 0.74902 1" />
-    </material>
-    <material name="yaskawa_silver">
-      <color rgba="0.75294 0.75294 0.75294 1" />
-    </material>
+    <xacro:macro name="material_yaskawa_blue">
+      <material name="${prefix}yaskawa_blue">
+        <color rgba="0.12941 0.12941 0.69020 1.0" />
+      </material>
+    </xacro:macro>
     <!-- link list -->
-    <!-- <link name="world" /> -->
     <link name="${prefix}base_link">
       <visual>
         <geometry>
-          <mesh filename="package://robot_planning/meshes/motomini/visual/base_link.stl" />
+          <mesh filename="package://robot_model/meshes/motomini/visual/base_link.stl" />
         </geometry>
-        <material name="yaskawa_blue" />
+        <xacro:material_yaskawa_blue />
       </visual>
       <collision>
         <geometry>
-          <mesh filename="package://robot_planning/meshes/motomini/collision/base_link.stl" />
+          <mesh
+            filename="package://robot_model/meshes/motomini/collision/base_link.stl" />
         </geometry>
       </collision>
@@ -26,11 +25,11 @@
       <visual>
         <geometry>
-          <mesh filename="package://robot_planning/meshes/motomini/visual/link_1_s.stl" />
+          <mesh filename="package://robot_model/meshes/motomini/visual/link_1_s.stl" />
         </geometry>
-        <material name="yaskawa_blue" />
+        <xacro:material_yaskawa_blue />
       </visual>
       <collision>
         <geometry>
-          <mesh filename="package://robot_planning/meshes/motomini/collision/link_1_s.stl" />
+          <mesh filename="package://robot_model/meshes/motomini/collision/link_1_s.stl" />
         </geometry>
       </collision>
@@ -39,11 +38,11 @@
       <visual>
         <geometry>
-          <mesh filename="package://robot_planning/meshes/motomini/visual/link_2_l.stl" />
+          <mesh filename="package://robot_model/meshes/motomini/visual/link_2_l.stl" />
         </geometry>
-        <material name="yaskawa_blue" />
+        <xacro:material_yaskawa_blue />
       </visual>
       <collision>
         <geometry>
-          <mesh filename="package://robot_planning/meshes/motomini/collision/link_2_l.stl" />
+          <mesh filename="package://robot_model/meshes/motomini/collision/link_2_l.stl" />
         </geometry>
       </collision>
@@ -52,11 +51,11 @@
       <visual>
         <geometry>
-          <mesh filename="package://robot_planning/meshes/motomini/visual/link_3_u.stl" />
+          <mesh filename="package://robot_model/meshes/motomini/visual/link_3_u.stl" />
         </geometry>
-        <material name="yaskawa_blue" />
+        <xacro:material_yaskawa_blue />
       </visual>
       <collision>
         <geometry>
-          <mesh filename="package://robot_planning/meshes/motomini/collision/link_3_u.stl" />
+          <mesh filename="package://robot_model/meshes/motomini/collision/link_3_u.stl" />
         </geometry>
       </collision>
@@ -65,11 +64,11 @@
       <visual>
         <geometry>
-          <mesh filename="package://robot_planning/meshes/motomini/visual/link_4_r.stl" />
+          <mesh filename="package://robot_model/meshes/motomini/visual/link_4_r.stl" />
         </geometry>
-        <material name="yaskawa_blue" />
+        <xacro:material_yaskawa_blue />
       </visual>
       <collision>
         <geometry>
-          <mesh filename="package://robot_planning/meshes/motomini/collision/link_4_r.stl" />
+          <mesh filename="package://robot_model/meshes/motomini/collision/link_4_r.stl" />
         </geometry>
       </collision>
@@ -78,11 +77,11 @@
       <visual>
         <geometry>
-          <mesh filename="package://robot_planning/meshes/motomini/visual/link_5_b.stl" />
+          <mesh filename="package://robot_model/meshes/motomini/visual/link_5_b.stl" />
         </geometry>
-        <material name="yaskawa_blue" />
+        <xacro:material_yaskawa_blue />
       </visual>
       <collision>
         <geometry>
-          <mesh filename="package://robot_planning/meshes/motomini/collision/link_5_b.stl" />
+          <mesh filename="package://robot_model/meshes/motomini/collision/link_5_b.stl" />
         </geometry>
       </collision>
@@ -91,11 +90,11 @@
       <visual>
         <geometry>
-          <mesh filename="package://robot_planning/meshes/motomini/visual/link_6_t.stl" />
+          <mesh filename="package://robot_model/meshes/motomini/visual/link_6_t.stl" />
         </geometry>
-        <material name="yaskawa_blue" />
+        <xacro:material_yaskawa_blue />
       </visual>
       <collision>
         <geometry>
-          <mesh filename="package://robot_planning/meshes/motomini/collision/link_6_t.stl" />
+          <mesh filename="package://robot_model/meshes/motomini/collision/link_6_t.stl" />
         </geometry>
       </collision>
@@ -104,9 +103,4 @@
     <!-- end of link list -->
     <!-- joint list -->
-    <!-- <joint name="world_base_link" type="fixed">
-      <parent link="world" />
-      <child link="${prefix}base_link" />
-      <origin xyz="0 0 0" rpy="0 0 0" />
-    </joint> -->
     <joint name="${prefix}joint_1_s" type="revolute">
       <parent link="${prefix}base_link" />

Commit message: tuning gui

File: motomini/urdf/motoman_motomini.urdf (robot description, URDF)
Before this commit: robot motoman_motomini, 10 links, 9 joints
Joints:
- joint workcell_joint: origin xyz=0.0 0.0 0.0 rpy=0 0 0 -> xyz=0.0 0.0 0.01 rpy=0 0 0

File: motomini/urdf/motoman_motomini_sensors.urdf.xacro (robot description, xacro)
@@ -16,5 +16,5 @@
     </link>
     <link name="world_range_link">
-        <visual>
+        <!-- <visual>
             <origin xyz="0.0 0.0 0.0" rpy="0.0 0.0 0.0" />
             <geometry>
@@ -27,5 +27,5 @@
                 <box size="0.3 0.06 0.03" />
             </geometry>
-        </collision>
+        </collision> -->
         <inertial>
             <mass value="0.05" />

Commit message: [feature] update the tracking

File: motomini/urdf/motoman_motomini.urdf (robot description, URDF)
Before this commit: robot motoman_motomini, 10 links, 9 joints
Links:
- link workcell: geometry visual mesh filename=package://motomini/meshes/motomini_workcell-Body.stl scale=0.001 0.001 0.001

Commit message: [feature] exactly collision debug

File: motomini/urdf/motoman_motomini.urdf (robot description, URDF)
Before this commit: robot motoman_motomini, 10 links, 9 joints
Links:
- link workcell: geometry collision mesh filename=package://motomini/meshes/motomini_workcell-Body.stl scale=0.001 0.001 0.001; visual mesh filename=package://motomini/meshes/motomini_workcell-Body.stl scale=0.001 0.001 0.001
