Commit message: [feature] collision bayesian optimizer
- Add bayes_optimize_collision.py: 4-phase TPE Bayesian optimizer for collision controller params
- Add run_collision_trial.py: single trial runner measuring penetration, force jitter, progress, tracking error
- Add collision_trial.yaml: trial config for collision optimizer
- Add tuning_results: best params, trial history CSVs
- Add docs/bayesian_optimization_theory.md: full theory doc (GP, TPE, cost functions)
- Update motomini.launch.py and URDF with collision support
- Update collision_debugger_node.cpp

Co-authored-by: Copilot <223556219+Copilot@users.noreply.github.com>

File: motomini/urdf/motoman_motomini_sensors.urdf.xacro (robot description, xacro)
@@ -15,5 +15,5 @@
         </inertial>
     </link>
-    <!-- <link name="test_obstacle">
+    <link name="test_obstacle">
         <visual>
             <geometry>
@@ -37,6 +37,6 @@
         <parent link="workcell" />
         <child link="test_obstacle" />
-        <origin xyz="0.27 -0.05 0.08" rpy="0 0 0" />
-    </joint> -->
+        <origin xyz="0.27 -0.05 -0.08" rpy="0 0 0" />
+    </joint>
     <joint name="world_depth_camera_joint" type="fixed">
         <parent link="workcell" />
