Commit message: [bug] collision box too big

File: motomini/urdf/motoman_motomini_sensors.urdf.xacro (robot description, xacro)
@@ -21,4 +21,9 @@
             </geometry>
         </visual>
+        <collision>
+            <geometry>
+                <cylinder radius="0.02" length="0.05" />
+            </geometry>
+        </collision>
         <inertial>
             <mass value="0.05" />
@@ -32,5 +37,5 @@
         <parent link="workcell" />
         <child link="world_range_link" />
-        <origin xyz="0.2 0.2 0.3" rpy="0 1.57142857143 0" />
+        <origin xyz="0.2 0.0 0.15" rpy="0 1.57142857143 0" />
     </joint>
     <joint name="world_depth_camera_joint" type="fixed">

Commit message: [bug] too slow and catesian joint crash

File: motomini/urdf/motoman_motomini_sensors.urdf.xacro (robot description, xacro)
@@ -17,18 +17,20 @@
     <link name="world_range_link">
         <visual>
+            <origin xyz="0.0 0.0 0.0" rpy="0.0 0.0 0.0" />
             <geometry>
-                <cylinder radius="0.02" length="0.05" />
+                <box size="0.05 0.05 0.05" />
             </geometry>
         </visual>
         <collision>
+            <origin xyz="0.0 0.0 0.0" rpy="0.0 0.0 0.0" />
             <geometry>
-                <cylinder radius="0.02" length="0.05" />
+                <box size="0.05 0.05 0.03" />
             </geometry>
         </collision>
         <inertial>
             <mass value="0.05" />
-            <origin xyz="0 0 0" />
-            <inertia ixx="0.0001" ixy="0" ixz="0"
-                iyy="0.0001" iyz="0"
+            <origin xyz="0.0 0.0 0.0" rpy="0.0 0.0 0.0" />
+            <inertia ixx="0.0001" ixy="0.0" ixz="0.0"
+                iyy="0.0001" iyz="0.0"
                 izz="0.0001" />
         </inertial>

File: motomini/urdf/motoman_motomini_tool.xacro (robot description, xacro)
@@ -51,5 +51,5 @@
         <visual>
           <!--visual_world_/Body.-->
-          <origin rpy="0 0 0" xyz="0.0 0.0 -0.045" />
+          <origin rpy="0 0 0" xyz="0.0 0.0 0" />
           <geometry>
             <mesh filename="package://motomini/meshes/tool-magnetic.dae" />
@@ -58,5 +58,5 @@
         <collision>
           <!--col__world__col_Body__BoundBox/col_Body__BoundBox.-->
-          <origin rpy="0 0 0" xyz="0.0 0.0 -0.045" />
+          <origin rpy="0 0 0" xyz="0.0 0.0 0" />
           <geometry>
             <mesh filename="package://motomini/meshes/tool-magnetic.dae" />
@@ -74,5 +74,5 @@
         <parent link="${parent_link}" />
         <child link="magnetic_link" />
-        <origin xyz="0 0 0.045" rpy="0 0 0" />
+        <origin xyz="0 0 0.045" rpy="3.1415926535897932384626433 0.0 0.0" />
       </joint>
     </xacro:if>

File: motomini/urdf/motoman_motomini_wrapper_realbot.urdf.xacro (robot description, xacro)
@@ -13,4 +13,5 @@
     <xacro:include filename="motoman_motomini_sensors.urdf.xacro" />
     <xacro:include filename="motoman_motomini_tool.xacro" />
+    <xacro:include filename="2axis.urdf.xacro" />
     <!-- ========= TOOLS ========= -->
     <xacro:motomini_tool
@@ -23,4 +24,9 @@
         <child link="workcell" />
         <origin xyz="0 0 0.068" rpy="0 0 0" />
+    </joint>
+    <joint name="world_to_gantry" type="fixed">
+        <parent link="world" />
+        <child link="gantry_base_link" />
+        <origin xyz="-0.05 -0.3 0.1" rpy="0 0 3.14" />
     </joint>
     <gazebo reference="link_1_s">

Commit message: workable check point

File: motomini/urdf/motoman_motomini_sensors.urdf.xacro (robot description, xacro)
@@ -19,13 +19,13 @@
             <origin xyz="0.0 0.0 0.0" rpy="0.0 0.0 0.0" />
             <geometry>
-                <box size="0.03 0.03 0.03" />
+                <box size="0.3 0.06 0.03" />
             </geometry>
         </visual>
-        <!-- <collision>
+        <collision>
             <origin xyz="0.0 0.0 0.0" rpy="0.0 0.0 0.0" />
             <geometry>
-                <box size="0.03 0.03 0.03" />
+                <box size="0.3 0.06 0.03" />
             </geometry>
-        </collision> -->
+        </collision>
         <inertial>
             <mass value="0.05" />
@@ -39,5 +39,5 @@
         <parent link="workcell" />
         <child link="world_range_link" />
-        <origin xyz="0.2 0.0 0.15" rpy="0 1.57142857143 0" />
+        <origin xyz="0.25 0.0 0.1" rpy="0 1.57142857143 0" />
     </joint>
     <joint name="world_depth_camera_joint" type="fixed">

Commit message: docs: add comprehensive README and update .gitignore for ROS2/Python/Tesseract project

File: motomini/urdf/motoman_motomini_sensors.urdf.xacro (robot description, xacro)
@@ -44,5 +44,5 @@
         <parent link="workcell" />
         <child link="world_depth_camera_link" />
-        <origin xyz="0.225 -0.225 0.245" rpy="0 3.14159 3.14159" />
+        <origin xyz="0.212 -0.027 0.496" rpy="0 3.14159 3.14159" />
     </joint>
     <gazebo reference="world_depth_camera_link">

File: motomini/urdf/motoman_motomini_tool.xacro (robot description, xacro)
@@ -104,5 +104,5 @@
         <parent link="${parent_link}" />
         <child link="calib_link" />
-        <origin xyz="0.0145 0.0 0.0455" rpy="-1.57 0 1.57" />
+        <origin xyz="0.0145 0.0 0.09" rpy="-1.57 0 1.57" />
       </joint>
     </xacro:if>

File: motomini/urdf/motoman_motomini_wrapper_realbot.urdf.xacro (robot description, xacro)
@@ -14,4 +14,5 @@
     <xacro:include filename="motoman_motomini_tool.xacro" />
     <xacro:include filename="2axis.urdf.xacro" />
+    <!-- <xacro:include filename="plate.urdf.xacro" /> -->
     <!-- ========= TOOLS ========= -->
     <xacro:motomini_tool
@@ -30,4 +31,9 @@
         <origin xyz="0.03 -0.46 0.0602" rpy="0 0 3.14" />
     </joint>
+    <!-- <joint name="world_to_plate" type="fixed">
+        <parent link="world" />
+        <child link="plate_body" />
+        <origin xyz="0.03 -0.46 0.0602" rpy="0 0 3.14" />
+    </joint> -->
     <gazebo reference="link_1_s">
         <turnGravityOff>true</turnGravityOff>

Commit message: [fix] multi thread

File: motomini/urdf/motoman_motomini_sensors.urdf.xacro (robot description, xacro)
@@ -15,34 +15,8 @@
         </inertial>
     </link>
-    <link name="world_range_link">
-        <!-- <visual>
-            <origin xyz="0.0 0.0 0.0" rpy="0.0 0.0 0.0" />
-            <geometry>
-                <box size="0.3 0.06 0.03" />
-            </geometry>
-        </visual>
-        <collision>
-            <origin xyz="0.0 0.0 0.0" rpy="0.0 0.0 0.0" />
-            <geometry>
-                <box size="0.3 0.06 0.03" />
-            </geometry>
-        </collision> -->
-        <inertial>
-            <mass value="0.05" />
-            <origin xyz="0.0 0.0 0.0" rpy="0.0 0.0 0.0" />
-            <inertia ixx="0.0001" ixy="0.0" ixz="0.0"
-                iyy="0.0001" iyz="0.0"
-                izz="0.0001" />
-        </inertial>
-    </link>
-    <joint name="world_range_joint" type="fixed">
-        <parent link="workcell" />
-        <child link="world_range_link" />
-        <origin xyz="0.25 0.0 0.1" rpy="0 1.57142857143 0" />
-    </joint>
     <joint name="world_depth_camera_joint" type="fixed">
         <parent link="workcell" />
         <child link="world_depth_camera_link" />
-        <origin xyz="0.212 -0.027 0.496" rpy="0 3.14159 3.14159" />
+        <origin xyz="0.212 -0.027 0.0" rpy="0 3.14159 1.57142857143" />
     </joint>
     <gazebo reference="world_depth_camera_link">

Commit message: [bug] oscillation with real_controller

File: motomini/urdf/motoman_motomini_sensors.urdf.xacro (robot description, xacro)
@@ -19,4 +19,31 @@
         <child link="world_depth_camera_link" />
         <origin xyz="0.212 -0.027 0.0" rpy="0 3.14159 1.57142857143" />
+    </joint>
+    <link name="obstacle">
+        <visual>
+            <geometry>
+                <box size="0.1 0.1 0.1"/>
+            </geometry>
+            <material>
+                <color rgba="0.8 0.2 0.2 1"/>
+            </material>
+        </visual>
+        <collision>
+            <geometry>
+                <box size="0.1 0.1 0.1"/>
+            </geometry>
+        </collision>
+        <inertial>
+            <mass value="1.0"/>
+            <origin xyz="0 0 0"/>
+            <inertia ixx="0.01" ixy="0" ixz="0"
+                     iyy="0.01" iyz="0"
+                     izz="0.01"/>
+        </inertial>
+    </link>
+    <joint name="obstacle_joint" type="fixed">
+        <parent link="workcell"/>
+        <child link="obstacle"/>
+        <origin xyz="0.5 0 0.05" rpy="0 0 0"/>
     </joint>
     <gazebo reference="world_depth_camera_link">

Commit message: [feature] sensor fillter

File: motomini/urdf/motoman_motomini_sensors.urdf.xacro (robot description, xacro)
@@ -15,35 +15,32 @@
         </inertial>
     </link>
+    <link name="test_obstacle">
+        <visual>
+            <geometry>
+                <box size="0.03 0.03 0.25" />
+            </geometry>
+        </visual>
+        <collision>
+            <geometry>
+                <box size="0.038 0.038 0.258" />
+            </geometry>
+        </collision>
+        <inertial>
+            <mass value="0.1" />
+            <origin xyz="0 0 0" />
+            <inertia ixx="0.001" ixy="0" ixz="0"
+                iyy="0.001" iyz="0"
+                izz="0.001" />
+        </inertial>
+    </link>
+    <joint name="obstacle_joint" type="fixed">
+        <parent link="workcell" />
+        <child link="test_obstacle" />
+        <origin xyz="0.27 -0.05 0.08" rpy="0 0 0" />
+    </joint>
     <joint name="world_depth_camera_joint" type="fixed">
         <parent link="workcell" />
         <child link="world_depth_camera_link" />
         <origin xyz="0.212 -0.027 0.0" rpy="0 3.14159 1.57142857143" />
-    </joint>
-    <link name="obstacle">
-        <visual>
-            <geometry>
-                <box size="0.1 0.1 0.1"/>
-            </geometry>
-            <material>
-                <color rgba="0.8 0.2 0.2 1"/>
-            </material>
-        </visual>
-        <collision>
-            <geometry>
-                <box size="0.1 0.1 0.1"/>
-            </geometry>
-        </collision>
-        <inertial>
-            <mass value="1.0"/>
-            <origin xyz="0 0 0"/>
-            <inertia ixx="0.01" ixy="0" ixz="0"
-                     iyy="0.01" iyz="0"
-                     izz="0.01"/>
-        </inertial>
-    </link>
-    <joint name="obstacle_joint" type="fixed">
-        <parent link="workcell"/>
-        <child link="obstacle"/>
-        <origin xyz="0.5 0 0.05" rpy="0 0 0"/>
     </joint>
     <gazebo reference="world_depth_camera_link">

Commit message: pose_track_vel_max

File: motomini/urdf/motoman_motomini_sensors.urdf.xacro (robot description, xacro)
@@ -15,5 +15,5 @@
         </inertial>
     </link>
-    <link name="test_obstacle">
+    <!-- <link name="test_obstacle">
         <visual>
             <geometry>
@@ -38,5 +38,5 @@
         <child link="test_obstacle" />
         <origin xyz="0.27 -0.05 0.08" rpy="0 0 0" />
-    </joint>
+    </joint> -->
     <joint name="world_depth_camera_joint" type="fixed">
         <parent link="workcell" />

Commit message: [feature] before force tunning

File: motomini/urdf/motoman_motomini_sensors.urdf.xacro (robot description, xacro)
@@ -15,5 +15,5 @@
         </inertial>
     </link>
-    <!-- <link name="test_obstacle">
+    <link name="test_obstacle">
         <visual>
             <geometry>
@@ -38,5 +38,5 @@
         <child link="test_obstacle" />
         <origin xyz="0.27 -0.05 0.08" rpy="0 0 0" />
-    </joint> -->
+    </joint>
     <joint name="world_depth_camera_joint" type="fixed">
         <parent link="workcell" />

Commit message: [feature] update image gui

File: motomini/urdf/motoman_motomini_sensors.urdf.xacro (robot description, xacro)
@@ -15,5 +15,5 @@
         </inertial>
     </link>
-    <link name="test_obstacle">
+    <!-- <link name="test_obstacle">
         <visual>
             <geometry>
@@ -38,9 +38,10 @@
         <child link="test_obstacle" />
         <origin xyz="0.27 -0.05 -0.08" rpy="0 0 0" />
-    </joint>
+    </joint> -->
     <joint name="world_depth_camera_joint" type="fixed">
         <parent link="workcell" />
         <child link="world_depth_camera_link" />
-        <origin xyz="0.212 -0.027 0.0" rpy="0 3.14159 1.57142857143" />
+        <!-- <origin xyz="0.212 -0.027 0.0" rpy="0 3.14159 1.57142857143" /> -->
+        <origin xyz="0.212 -0.027 0.0" rpy="0 0 1.57142857143" />
     </joint>
     <gazebo reference="world_depth_camera_link">

Commit message: [feature] none singularity

File: motomini/urdf/motoman_motomini_sensors.urdf.xacro (robot description, xacro)
@@ -15,13 +15,13 @@
         </inertial>
     </link>
-    <!-- <link name="test_obstacle">
+    <link name="test_obstacle">
         <visual>
             <geometry>
-                <box size="0.03 0.03 0.25" />
+                <cylinder radius="0.015" length="0.25" />
             </geometry>
         </visual>
         <collision>
             <geometry>
-                <box size="0.038 0.038 0.258" />
+                <cylinder radius="0.019" length="0.258" />
             </geometry>
         </collision>
@@ -38,5 +38,5 @@
         <child link="test_obstacle" />
         <origin xyz="0.27 -0.05 -0.08" rpy="0 0 0" />
-    </joint> -->
+    </joint>
     <joint name="world_depth_camera_joint" type="fixed">
         <parent link="workcell" />

Commit message: [update] seperate controller

File: motomini/urdf/motoman_motomini_sensors.urdf.xacro (robot description, xacro)
@@ -15,5 +15,5 @@
         </inertial>
     </link>
-    <link name="test_obstacle">
+    <!-- <link name="test_obstacle">
         <visual>
             <geometry>
@@ -37,6 +37,6 @@
         <parent link="workcell" />
         <child link="test_obstacle" />
-        <origin xyz="0.27 -0.05 -0.08" rpy="0 0 0" />
-    </joint>
+        <origin xyz="0.27 -0.05 0.1" rpy="0 0 0" />
+    </joint> -->
     <joint name="world_depth_camera_joint" type="fixed">
         <parent link="workcell" />

Commit message: [bug] non stop

File: motomini/urdf/motoman_motomini_sensors.urdf.xacro (robot description, xacro)
@@ -15,5 +15,5 @@
         </inertial>
     </link>
-    <link name="test_obstacle">
+    <!-- <link name="test_obstacle">
         <visual>
             <geometry>
@@ -38,5 +38,5 @@
         <child link="test_obstacle" />
         <origin xyz="0.26 -0.05 0.01" rpy="0 1.579 0" />
-    </joint>
+    </joint> -->
     <joint name="world_depth_camera_joint" type="fixed">
         <parent link="workcell" />
