Commit message: [feature] gandtry

File: motomini/urdf/2axis.urdf.xacro (robot description, xacro)
@@ -37,4 +37,12 @@
       </geometry>
     </collision>
+  </link>
+  <link name='working_tip'>
+    <visual>
+      <origin xyz="0.0 0.0 -0.025" rpy="0.0 0.0 3.14" />
+      <geometry>
+        <box size="0.01 0.01 0.05" />
+      </geometry>
+    </visual>
   </link>
   <!-- Joint 1: Prismatic movement along the X-axis (1 0 0) -->
@@ -93,4 +101,9 @@
     </collision>
   </link>
+  <joint name="working_tip_tool" type="fixed">
+    <parent link="gantry_tool_link" />
+    <child link="working_tip" />
+    <origin xyz="0.0 -0.07 0.05" rpy="0.0 0.0 0.0" />
+  </joint>
   <!-- Fixed joint attaching the tool to the bottom of the Z-shaft -->
   <joint name="gantry_tool_joint" type="fixed">

File: motomini/urdf/motoman_motomini.srdf.xacro (robot description, xacro)
@@ -19,4 +19,7 @@
         <chain base_link="base_link" tip_link="${actual_tip_link}" />
     </group>
+    <group name="gantry">
+        <chain base_link="gantry_base_link" tip_link="gantry_tool_link" />
+    </group>
     <group_state name="home" group="manipulator">
         <joint name="joint_1_s" value="0" />
@@ -26,4 +29,8 @@
         <joint name="joint_5_b" value="0" />
         <joint name="joint_6_t" value="0" />
+    </group_state>
+    <group_state name="home" group="gantry">
+        <joint name="joint_x" value="0" />
+        <joint name="joint_z" value="0" />
     </group_state>
     <kinematics_plugin_config
@@ -49,4 +56,7 @@
     <disable_collisions link1="workcell" link2="link_1_s" reason="Mounted" />
     <disable_collisions link1="workcell" link2="link_2_l" reason="Workcell Mount" />
+    <disable_collisions link1="gantry_base_link" link2="x_carriage" reason="Adjacent" />
+    <disable_collisions link1="x_carriage" link2="z_shaft" reason="Adjacent" />
+    <disable_collisions link1="z_shaft" link2="gantry_tool_link" reason="Adjacent" />
     <!-- <disable_collisions link1="workcell" link2="magnetic_link" reason="Workcell Mount" /> -->
     <xacro:if value="${tool_type == 'gripper'}">

File: motomini/urdf/motoman_motomini_sensors.urdf.xacro (robot description, xacro)
@@ -19,5 +19,5 @@
             <origin xyz="0.0 0.0 0.0" rpy="0.0 0.0 0.0" />
             <geometry>
-                <box size="0.05 0.05 0.05" />
+                <box size="0.03 0.03 0.03" />
             </geometry>
         </visual>
@@ -25,5 +25,5 @@
             <origin xyz="0.0 0.0 0.0" rpy="0.0 0.0 0.0" />
             <geometry>
-                <box size="0.05 0.05 0.03" />
+                <box size="0.03 0.03 0.03" />
             </geometry>
         </collision>

Commit message: [feature] slow tracking

File: motomini/urdf/2axis.urdf.xacro (robot description, xacro)
@@ -13,10 +13,10 @@
       </material>
     </visual>
-    <collision>
+    <!-- <collision>
       <origin xyz="0.14 0 0" rpy="0 0 0" />
       <geometry>
         <box size="0.35 0.1 0.05" />
       </geometry>
-    </collision>
+    </collision> -->
   </link>
   <!-- ================= LINK 1 (X-Axis Carriage) ================= -->
@@ -31,10 +31,10 @@
       </material>
     </visual>
-    <collision>
+    <!-- <collision>
       <origin xyz="0 0 0.05" rpy="0 0 0" />
       <geometry>
         <box size="0.08 0.08 0.08" />
       </geometry>
-    </collision>
+    </collision> -->
   </link>
   <link name='working_tip'>
@@ -66,10 +66,10 @@
       </material>
     </visual>
-    <collision>
+    <!-- <collision>
       <origin xyz="0 0 -0.05" rpy="0 0 0" />
       <geometry>
         <box size="0.04 0.04 0.15" />
       </geometry>
-    </collision>
+    </collision> -->
   </link>
   <!-- Joint 2: Prismatic movement along the Z-axis (0 0 1) -->
@@ -94,10 +94,10 @@
       </material>
     </visual>
-    <collision>
+    <!-- <collision>
       <origin xyz="0 0 -0.05" rpy="0 0 0" />
       <geometry>
         <box size="0.04 0.04 0.15" />
       </geometry>
-    </collision>
+    </collision> -->
   </link>
   <joint name="working_tip_tool" type="fixed">

File: motomini/urdf/motoman_motomini_sensors.urdf.xacro (robot description, xacro)
@@ -22,10 +22,10 @@
             </geometry>
         </visual>
-        <collision>
+        <!-- <collision>
             <origin xyz="0.0 0.0 0.0" rpy="0.0 0.0 0.0" />
             <geometry>
                 <box size="0.03 0.03 0.03" />
             </geometry>
-        </collision>
+        </collision> -->
         <inertial>
             <mass value="0.05" />

Commit message: [fix] tracking period

File: motomini/urdf/2axis.urdf.xacro (robot description, xacro)
@@ -40,9 +40,17 @@
   <link name='working_tip'>
     <visual>
+      <origin xyz="0.0 0.0 0.0" rpy="0.0 3.14 0.0" />
+      <geometry>
+        <mesh
+          filename="package://motomini/meshes/gantry/gantry-tool.stl"
+          scale="0.001 0.001 0.001" />
+      </geometry>
+    </visual>
+    <!-- <visual>
       <origin xyz="0.0 0.0 -0.025" rpy="0.0 0.0 3.14" />
       <geometry>
         <box size="0.01 0.01 0.05" />
       </geometry>
-    </visual>
+    </visual> -->
   </link>
   <!-- Joint 1: Prismatic movement along the X-axis (1 0 0) -->
@@ -86,7 +94,9 @@
   <link name="gantry_tool_link">
     <visual>
-      <origin xyz="0 -0.03 0.0" rpy="0 0 0" />
+      <origin xyz="0 -0.07 0.0" rpy="0 0 3.14" />
       <geometry>
-        <box size="0.02 0.1 0.01" />
+        <mesh
+          filename="package://motomini/meshes/gantry/gantry-hand.stl"
+          scale="0.001 0.001 0.001" />
       </geometry>
       <material name="red">
@@ -104,5 +114,6 @@
     <parent link="gantry_tool_link" />
     <child link="working_tip" />
-    <origin xyz="0.0 -0.07 0.05" rpy="0.0 0.0 0.0" />
+    <origin xyz="0.0 -0.1451 0.05" rpy="0.0 0.0 3.14" />
+    <!-- <origin xyz="0.0 -0.1451 0.133" rpy="0.0 0.0 3.14" /> -->
   </joint>
   <!-- Fixed joint attaching the tool to the bottom of the Z-shaft -->

File: motomini/urdf/motoman_motomini.urdf (robot description, URDF)
Before this commit: robot motoman_motomini, 10 links, 9 joints
Joints:
- joint joint_1_s: limit lower=-2.967 upper=2.967 effort=50.0 velocity=0.5 -> lower=-2.9670 upper=2.9670 effort=0.12 velocity=5.4977
- joint joint_2_l: limit lower=-1.4835 upper=1.5707 effort=50.0 velocity=0.5 -> lower=-1.4835 upper=1.5707 effort=0.12 velocity=5.4977
- joint joint_3_u: limit lower=-0.8726 upper=1.5707 effort=50.0 velocity=0.5 -> lower=-0.8726 upper=1.5707 effort=0.12 velocity=7.3304
- joint joint_4_r: limit lower=-2.4434 upper=2.4434 effort=50.0 velocity=0.5 -> lower=-2.4434 upper=2.4434 effort=0.07 velocity=10.4719
- joint joint_5_b: limit lower=-0.5235 upper=3.6651 effort=50.0 velocity=0.5 -> lower=-0.5235 upper=3.6651 effort=0.07 velocity=10.4719
- joint joint_6_t: limit lower=-6.2831 upper=6.2831 effort=50.0 velocity=0.5 -> lower=-6.2831 upper=6.2831 effort=0.07 velocity=10.4719

File: motomini/urdf/motoman_motomini_wrapper_realbot.urdf.xacro (robot description, xacro)
@@ -28,5 +28,5 @@
         <parent link="world" />
         <child link="gantry_base_link" />
-        <origin xyz="-0.05 -0.3 0.1" rpy="0 0 3.14" />
+        <origin xyz="0.03 -0.46 0.0602" rpy="0 0 3.14" />
     </joint>
     <gazebo reference="link_1_s">

Commit message: [bug] no optimal controller

File: motomini/urdf/2axis.urdf.xacro (robot description, xacro)
@@ -114,5 +114,5 @@
     <parent link="gantry_tool_link" />
     <child link="working_tip" />
-    <origin xyz="0.0 -0.1451 0.05" rpy="0.0 0.0 3.14" />
+    <origin xyz="0.0 -0.1451 0.045" rpy="0.0 0.0 3.14" />
     <!-- <origin xyz="0.0 -0.1451 0.133" rpy="0.0 0.0 3.14" /> -->
   </joint>

File: motomini/urdf/motoman_motomini_sensors.urdf.xacro (robot description, xacro)
@@ -15,13 +15,13 @@
         </inertial>
     </link>
-    <!-- <link name="test_obstacle">
+    <link name="test_obstacle">
         <visual>
             <geometry>
-                <cylinder radius="0.015" length="0.25" />
+                <cylinder radius="0.03" length="0.08" />
             </geometry>
         </visual>
         <collision>
             <geometry>
-                <cylinder radius="0.019" length="0.258" />
+                <cylinder radius="0.03" length="0.08" />
             </geometry>
         </collision>
@@ -37,6 +37,6 @@
         <parent link="workcell" />
         <child link="test_obstacle" />
-        <origin xyz="0.27 -0.05 0.1" rpy="0 0 0" />
-    </joint> -->
+        <origin xyz="0.26 -0.05 0.01" rpy="0 1.579 0" />
+    </joint>
     <joint name="world_depth_camera_joint" type="fixed">
         <parent link="workcell" />

File: motomini/urdf/motoman_motomini_wrapper_realbot.urdf.xacro (robot description, xacro)
@@ -29,5 +29,5 @@
         <parent link="world" />
         <child link="gantry_base_link" />
-        <origin xyz="0.03 -0.46 0.0602" rpy="0 0 3.14" />
+        <origin xyz="0.07 -0.465 0.0602" rpy="0 0 3.14" />
     </joint>
     <!-- <joint name="world_to_plate" type="fixed">
